Commit message: Update robots and arena to final version, rename test.launch to arena.launch, add arena_no_gui.launch which launches without gui

File: urdf/ball.gazebo.xacro (robot description, xacro)
@@ -4,7 +4,7 @@
         <mu1>10</mu1>
         <mu2>1</mu2>
-        <kp>500.0</kp>
-        <kd>100</kd>
-        <minDepth>.001</minDepth>
+        <kp>5000.0</kp>
+        <kd>0</kd>
+        <minDepth>0</minDepth>
         <maxVel>1000</maxVel>
         <material>Gazebo/Red</material>
@@ -21,3 +21,23 @@
         </surface> -->
     </gazebo>
+    <gazebo reference="extra">
+        <mu1>10</mu1>
+        <mu2>1</mu2>
+        <kp>5000.0</kp>
+        <kd>0</kd>
+        <minDepth>0</minDepth>
+        <maxVel>0.1</maxVel>
+        <material>Gazebo/Red</material>
+        <!-- <surface>
+            <bounce>
+                <restitution_coefficient>.5</restitution_coefficient>
+                <threshold>0.01</threshold>
+            </bounce>
+            <contact>
+                <ode>
+                    <max_vel>100000</max_vel>
+                </ode>
+            </contact>
+        </surface> -->
+    </gazebo>
 </robot>

File: urdf/ball.urdf.xacro (robot description, xacro)
@@ -25,3 +25,31 @@
         </inertial>
     </link>
+    <link name="extra">
+        <visual>
+            <origin xyz="0 0 0" rpy="0 0 0"/>
+            <geometry>
+                <sphere radius=".2"/>
+            </geometry>
+            <material name="red"/>
+        </visual>
+        <collision>
+            <origin xyz="0 0 0" rpy="0 0 0"/>
+            <geometry>
+                <sphere radius=".2"/>
+            </geometry>
+        </collision>
+        <inertial>
+            <origin xyz="0 0 0" rpy="0 0 0"/>
+            <mass value="1.3729096e+00"/>
+            <inertia ixx="8.7002718e-03" ixy="-4.7576583e-05" ixz="1.1160499e-04"
+                 iyy="8.6195418e-03" iyz="-3.5422299e-06"
+                 izz="1.4612727e-02" />
+        </inertial>
+    </link>
+    <joint name="extra_joint" type="continuous">
+        <parent link="base_link"/>
+        <child link="extra"/>
+        <origin xyz="0.0 0.144 0.023" rpy="-1.57 0 0"/>
+        <axis xyz="0 0 1"/>
+    </joint>
 </robot>

File: urdf/turtle.urdf.xacro (robot description, xacro)
@@ -17,5 +17,5 @@
       <origin xyz="-0.064 0 0.047" rpy="0 0 0"/>
       <geometry>
-        <box size="0.3 0.3 0.094"/>
+        <cylinder radius="0.15" length="0.1"/>
       </geometry>
       <material name="light_black"/>
@@ -24,5 +24,5 @@
       <origin xyz="-0.064 0 0.047" rpy="0 0 0"/>
       <geometry>
-        <box size="0.4 0.4 0.094"/>
+        <cylinder radius="0.15" length="0.1"/>
       </geometry>
     </collision>
@@ -43,7 +43,7 @@
   <link name="wheel_left_link">
     <visual>
-      <origin xyz="0 0 0" rpy="1.57 0 0"/>
-      <geometry>
-        <mesh filename="package://turtlebot3_description/meshes/wheels/left_tire.stl" scale="0.001 0.001 0.001"/>
+      <origin xyz="0 0 0" rpy="0 0 0"/>
+      <geometry>
+        <cylinder length="0.018" radius="0.033"/>
       </geometry>
       <material name="dark"/>
@@ -57,5 +57,5 @@
     <inertial>
       <origin xyz="0 0 0" />
-      <mass value="2.8498940e-02" />
+      <mass value="1" />
       <inertia ixx="1.1175580e-05" ixy="-4.2369783e-11" ixz="-5.9381719e-09"
                iyy="1.1192413e-05" iyz="-1.4400107e-11"
@@ -71,7 +71,7 @@
   <link name="wheel_right_link">
     <visual>
-      <origin xyz="0 0 0" rpy="1.57 0 0"/>
-      <geometry>
-        <mesh filename="package://turtlebot3_description/meshes/wheels/right_tire.stl" scale="0.001 0.001 0.001"/>
+      <origin xyz="0 0 0" rpy="0 0 0"/>
+      <geometry>
+        <cylinder length="0.018" radius="0.033"/>
       </geometry>
       <material name="dark"/>
@@ -85,5 +85,5 @@
     <inertial>
       <origin xyz="0 0 0" />
-      <mass value="2.8498940e-02" />
+      <mass value="1" />
       <inertia ixx="1.1175580e-05" ixy="-4.2369783e-11" ixz="-5.9381719e-09"
                iyy="1.1192413e-05" iyz="-1.4400107e-11"
@@ -105,5 +105,5 @@
     <inertial>
       <origin xyz="0 0 0" />
-      <mass value="0.005" />
+      <mass value="1" />
       <inertia ixx="0.001" ixy="0.0" ixz="0.0"
                iyy="0.001" iyz="0.0"
@@ -125,5 +125,5 @@
     <inertial>
       <origin xyz="0 0 0" />
-      <mass value="0.005" />
+      <mass value="1" />
       <inertia ixx="0.001" ixy="0.0" ixz="0.0"
                iyy="0.001" iyz="0.0"
@@ -143,5 +143,5 @@
   </joint>
   <link name="base_scan">
-    <visual>
+    <!-- <visual>
       <origin xyz="0 0 0" rpy="0 0 0"/>
       <geometry>
@@ -149,5 +149,5 @@
       </geometry>
       <material name="dark"/>
-    </visual>
+    </visual> -->
     <collision>
       <origin xyz="0.015 0 -0.0065" rpy="0 0 0"/>
@@ -170,10 +170,10 @@
   </joint>
   <link name="camera_link">
-    <visual>
+    <!-- <visual>
      <origin xyz="0 0 0" rpy="1.57 0 1.57"/>
       <geometry>
        <mesh filename="package://turtlebot3_description/meshes/sensors/r200.dae" />
       </geometry>
-    </visual>
+    </visual> -->
     <collision>
       <origin xyz="0.003 0.065 0.007" rpy="0 0 0"/>

File: urdf/turtlebot3_waffle.gazebo.xacro (robot description, xacro)
@@ -6,19 +6,14 @@
   <gazebo reference="base_link">
     <material>Gazebo/DarkGrey</material>
-    <surface>
-      <bounce>
-        <restitution_coefficient>1</restitution_coefficient>
-        <threshold>0</threshold>
-      </bounce>
-      <contact>
-        <ode>
-          <max_vel>100000</max_vel>
-        </ode>
-      </contact>
-    </surface>
+    <mu1>1</mu1>
+    <mu2>1</mu2>
+    <kp>1000000</kp>
+    <kd>0</kd>
+    <minDepth>0</minDepth>
+    <maxVel>1000</maxVel>
   </gazebo>
   <gazebo reference="wheel_left_link">
     <mu1>10</mu1>
-    <mu2>1</mu2>
+    <mu2>.5</mu2>
     <kp>500000.0</kp>
     <kd>10.0</kd>
@@ -30,7 +25,7 @@
   <gazebo reference="wheel_right_link">
     <mu1>10</mu1>
-    <mu2>1</mu2>
+    <mu2>.5</mu2>
     <kp>500000.0</kp>
-    <kd>10.0</kd>
+    <kd>10</kd>
     <minDepth>0.001</minDepth>
     <maxVel>0.01</maxVel>
@@ -39,6 +34,6 @@
   </gazebo>
   <gazebo reference="caster_back_right_link">
-    <mu1>0</mu1>
-    <mu2>0</mu2>
+    <mu1>.5</mu1>
+    <mu2>.5</mu2>
     <kp>1000000.0</kp>
     <kd>100.0</kd>
@@ -48,6 +43,6 @@
   </gazebo>
   <gazebo reference="caster_back_left_link">
-    <mu1>0</mu1>
-    <mu2>0.</mu2>
+    <mu1>.5</mu1>
+    <mu2>.5</mu2>
     <kp>1000000.0</kp>
     <kd>100.0</kd>
