Commit message: Use waffle, add ball test, add single agent test, all launch, urdf, or world files

File: urdf/turtle.urdf.xacro (robot description, xacro)
@@ -15,7 +15,7 @@
   <link name="base_link">
     <visual>
-      <origin xyz="-0.064 0 0.0" rpy="0 0 0"/>
-      <geometry>
-        <mesh filename="package://turtlebot3_description/meshes/bases/waffle_base.stl" scale="0.001 0.001 0.001"/>
+      <origin xyz="-0.064 0 0.047" rpy="0 0 0"/>
+      <geometry>
+        <box size="0.3 0.3 0.094"/>
       </geometry>
       <material name="light_black"/>
@@ -24,5 +24,5 @@
       <origin xyz="-0.064 0 0.047" rpy="0 0 0"/>
       <geometry>
-        <box size="0.266 0.266 0.094"/>
+        <box size="0.4 0.4 0.094"/>
       </geometry>
     </collision>

File: urdf/turtlebot3_waffle.gazebo.xacro (robot description, xacro)
@@ -6,41 +6,52 @@
   <gazebo reference="base_link">
     <material>Gazebo/DarkGrey</material>
+    <surface>
+      <bounce>
+        <restitution_coefficient>1</restitution_coefficient>
+        <threshold>0</threshold>
+      </bounce>
+      <contact>
+        <ode>
+          <max_vel>100000</max_vel>
+        </ode>
+      </contact>
+    </surface>
   </gazebo>
   <gazebo reference="wheel_left_link">
-    <mu1>0.1</mu1>
-    <mu2>0.1</mu2>
+    <mu1>10</mu1>
+    <mu2>1</mu2>
     <kp>500000.0</kp>
     <kd>10.0</kd>
     <minDepth>0.001</minDepth>
-    <maxVel>0.1</maxVel>
+    <maxVel>0.01</maxVel>
     <fdir1>1 0 0</fdir1>
     <material>Gazebo/FlatBlack</material>
   </gazebo>
   <gazebo reference="wheel_right_link">
-    <mu1>0.1</mu1>
-    <mu2>0.1</mu2>
+    <mu1>10</mu1>
+    <mu2>1</mu2>
     <kp>500000.0</kp>
     <kd>10.0</kd>
     <minDepth>0.001</minDepth>
-    <maxVel>0.1</maxVel>
+    <maxVel>0.01</maxVel>
     <fdir1>1 0 0</fdir1>
     <material>Gazebo/FlatBlack</material>
   </gazebo>
   <gazebo reference="caster_back_right_link">
-    <mu1>0.1</mu1>
-    <mu2>0.1</mu2>
+    <mu1>0</mu1>
+    <mu2>0</mu2>
     <kp>1000000.0</kp>
     <kd>100.0</kd>
     <minDepth>0.001</minDepth>
-    <maxVel>1.0</maxVel>
+    <maxVel>0.01</maxVel>
     <material>Gazebo/FlatBlack</material>
   </gazebo>
   <gazebo reference="caster_back_left_link">
-    <mu1>0.1</mu1>
-    <mu2>0.1</mu2>
+    <mu1>0</mu1>
+    <mu2>0.</mu2>
     <kp>1000000.0</kp>
     <kd>100.0</kd>
     <minDepth>0.001</minDepth>
-    <maxVel>1.0</maxVel>
+    <maxVel>0.01</maxVel>
     <material>Gazebo/FlatBlack</material>
   </gazebo>
@@ -69,6 +80,6 @@
       <wheelSeparation>0.287</wheelSeparation>
       <wheelDiameter>0.066</wheelDiameter>
-      <wheelAcceleration>1</wheelAcceleration>
-      <wheelTorque>10</wheelTorque>
+      <wheelAcceleration>100</wheelAcceleration>
+      <wheelTorque>100</wheelTorque>
       <rosDebugLevel>na</rosDebugLevel>
     </plugin>

Commit message: Edit URDF files for maximum efficiency

File: urdf/turtle.urdf.xacro (robot description, xacro)
@@ -42,5 +42,5 @@
   </joint>
   <link name="wheel_left_link">
-    <visual>
+    <!-- <visual>
       <origin xyz="0 0 0" rpy="0 0 0"/>
       <geometry>
@@ -48,5 +48,5 @@
       </geometry>
       <material name="dark"/>
-    </visual>
+    </visual> -->
     <collision>
       <origin xyz="0 0 0" rpy="0 0 0"/>
@@ -61,5 +61,5 @@
                iyy="1.1192413e-05" iyz="-1.4400107e-11"
                izz="2.0712558e-05" />
-      </inertial>
+    </inertial>
   </link>
   <joint name="wheel_right_joint" type="continuous">
@@ -70,5 +70,5 @@
   </joint>
   <link name="wheel_right_link">
-    <visual>
+    <!-- <visual>
       <origin xyz="0 0 0" rpy="0 0 0"/>
       <geometry>
@@ -76,5 +76,5 @@
       </geometry>
       <material name="dark"/>
-    </visual>
+    </visual> -->
     <collision>
       <origin xyz="0 0 0" rpy="0 0 0"/>
@@ -89,5 +89,5 @@
                iyy="1.1192413e-05" iyz="-1.4400107e-11"
                izz="2.0712558e-05" />
-      </inertial>
+    </inertial>
   </link>
   <joint name="caster_back_right_joint" type="fixed">
@@ -131,17 +131,17 @@
     </inertial>
   </link>
-  <joint name="imu_joint" type="fixed">
+  <!-- <joint name="imu_joint" type="fixed">
     <parent link="base_link"/>
     <child link="imu_link"/>
     <origin xyz="0.0 0 0.068" rpy="0 0 0"/>
   </joint>
-  <link name="imu_link"/>
-  <joint name="scan_joint" type="fixed">
+  <link name="imu_link"/> -->
+  <!-- <joint name="scan_joint" type="fixed">
     <parent link="base_link"/>
     <child link="base_scan"/>
     <origin xyz="-0.064 0 0.122" rpy="0 0 0"/>
-  </joint>
-  <link name="base_scan">
-    <!-- <visual>
+  </joint> -->
+  <!-- <link name="base_scan">
+    <visual>
       <origin xyz="0 0 0" rpy="0 0 0"/>
       <geometry>
@@ -149,5 +149,5 @@
       </geometry>
       <material name="dark"/>
-    </visual> -->
+    </visual>
     <collision>
       <origin xyz="0.015 0 -0.0065" rpy="0 0 0"/>
@@ -163,6 +163,6 @@
                izz="0.001" />
     </inertial>
-  </link>
-  <joint name="camera_joint" type="fixed">
+  </link> -->
+  <!-- <joint name="camera_joint" type="fixed">
     <origin xyz="0.064 -0.065 0.094" rpy="0 0 0"/>
     <parent link="base_link"/>
@@ -170,10 +170,10 @@
   </joint>
   <link name="camera_link">
-    <!-- <visual>
+    <visual>
      <origin xyz="0 0 0" rpy="1.57 0 1.57"/>
       <geometry>
        <mesh filename="package://turtlebot3_description/meshes/sensors/r200.dae" />
       </geometry>
-    </visual> -->
+    </visual>
     <collision>
       <origin xyz="0.003 0.065 0.007" rpy="0 0 0"/>
@@ -182,6 +182,6 @@
       </geometry>
     </collision>
-    <!-- This inertial field needs doesn't contain reliable data!! -->
-<!--   <inertial>
+    This inertial field needs doesn't contain reliable data!!
+  <inertial>
       <mass value="0.564" />
       <origin xyz="0 0 0" />
@@ -189,5 +189,5 @@
                iyy="0.000498940" iyz="0.0"
                izz="0.003879257" />
-    </inertial>-->
+    </inertial>
   </link>
   <joint name="camera_rgb_joint" type="fixed">
@@ -214,4 +214,4 @@
     <child link="camera_depth_optical_frame"/>
   </joint>
-  <link name="camera_depth_optical_frame"/>
+  <link name="camera_depth_optical_frame"/> -->
 </robot>

File: urdf/turtlebot3_waffle.gazebo.xacro (robot description, xacro)
@@ -51,5 +51,5 @@
     <material>Gazebo/FlatBlack</material>
   </gazebo>
-  <gazebo reference="imu_link">
+  <!-- <gazebo reference="imu_link">
     <sensor type="imu" name="imu">
       <always_on>true</always_on>
@@ -57,5 +57,5 @@
     </sensor>
     <material>Gazebo/Grey</material>
-  </gazebo>
+  </gazebo> -->
   <gazebo>
     <plugin name="turtlebot3_waffle_controller" filename="libgazebo_ros_diff_drive.so">
@@ -80,5 +80,5 @@
     </plugin>
   </gazebo>
-  <gazebo>
+  <!-- <gazebo>
     <plugin name="imu_plugin" filename="libgazebo_ros_imu.so">
       <alwaysOn>true</alwaysOn>
@@ -107,5 +107,5 @@
       </imu>
     </plugin>
-  </gazebo>
+  </gazebo> -->
   <!-- <gazebo reference="base_scan">
     <material>Gazebo/FlatBlack</material>

Commit message: Adds 350 gen run, urdf modifications, and world file modification for visualized simulation

File: urdf/turtle.urdf.xacro (robot description, xacro)
@@ -42,5 +42,5 @@
   </joint>
   <link name="wheel_left_link">
-    <!-- <visual>
+    <visual>
       <origin xyz="0 0 0" rpy="0 0 0"/>
       <geometry>
@@ -48,5 +48,5 @@
       </geometry>
       <material name="dark"/>
-    </visual> -->
+    </visual>
     <collision>
       <origin xyz="0 0 0" rpy="0 0 0"/>
@@ -70,5 +70,5 @@
   </joint>
   <link name="wheel_right_link">
-    <!-- <visual>
+    <visual>
       <origin xyz="0 0 0" rpy="0 0 0"/>
       <geometry>
@@ -76,5 +76,5 @@
       </geometry>
       <material name="dark"/>
-    </visual> -->
+    </visual>
     <collision>
       <origin xyz="0 0 0" rpy="0 0 0"/>

Commit message: Updates to final version of world and urdf files

File: urdf/turtle.urdf.xacro (robot description, xacro)
@@ -131,16 +131,16 @@
     </inertial>
   </link>
-  <!-- <joint name="imu_joint" type="fixed">
+  <joint name="imu_joint" type="fixed">
     <parent link="base_link"/>
     <child link="imu_link"/>
     <origin xyz="0.0 0 0.068" rpy="0 0 0"/>
   </joint>
-  <link name="imu_link"/> -->
-  <!-- <joint name="scan_joint" type="fixed">
+  <link name="imu_link"/>
+  <joint name="scan_joint" type="fixed">
     <parent link="base_link"/>
     <child link="base_scan"/>
     <origin xyz="-0.064 0 0.122" rpy="0 0 0"/>
-  </joint> -->
-  <!-- <link name="base_scan">
+  </joint>
+  <link name="base_scan">
     <visual>
       <origin xyz="0 0 0" rpy="0 0 0"/>
@@ -163,6 +163,6 @@
                izz="0.001" />
     </inertial>
-  </link> -->
-  <!-- <joint name="camera_joint" type="fixed">
+  </link>
+  <joint name="camera_joint" type="fixed">
     <origin xyz="0.064 -0.065 0.094" rpy="0 0 0"/>
     <parent link="base_link"/>
@@ -182,5 +182,5 @@
       </geometry>
     </collision>
-    This inertial field needs doesn't contain reliable data!!
+  <!-- This inertial field needs doesn't contain reliable data!! -->
   <inertial>
       <mass value="0.564" />
@@ -214,4 +214,4 @@
     <child link="camera_depth_optical_frame"/>
   </joint>
-  <link name="camera_depth_optical_frame"/> -->
+  <link name="camera_depth_optical_frame"/>
 </robot>

File: urdf/turtlebot3_waffle.gazebo.xacro (robot description, xacro)
@@ -51,5 +51,5 @@
     <material>Gazebo/FlatBlack</material>
   </gazebo>
-  <!-- <gazebo reference="imu_link">
+  <gazebo reference="imu_link">
     <sensor type="imu" name="imu">
       <always_on>true</always_on>
@@ -57,5 +57,5 @@
     </sensor>
     <material>Gazebo/Grey</material>
-  </gazebo> -->
+  </gazebo>
   <gazebo>
     <plugin name="turtlebot3_waffle_controller" filename="libgazebo_ros_diff_drive.so">
@@ -80,5 +80,5 @@
     </plugin>
   </gazebo>
-  <!-- <gazebo>
+  <gazebo>
     <plugin name="imu_plugin" filename="libgazebo_ros_imu.so">
       <alwaysOn>true</alwaysOn>
@@ -107,6 +107,6 @@
       </imu>
     </plugin>
-  </gazebo> -->
-  <!-- <gazebo reference="base_scan">
+  </gazebo>
+  <gazebo reference="base_scan">
     <material>Gazebo/FlatBlack</material>
     <sensor type="ray" name="lds_lfcd_sensor">
@@ -182,4 +182,4 @@
       </plugin>
     </sensor>
-  </gazebo> -->
+  </gazebo>
 </robot>
